File: MedidoPump.kicad_pcb (KiCad board)
At the start: 2 copper layers, 165.1 x 101.6 mm, 46 parts, among them J1 Flow_Fwd, J2 Flow_Rev, J3 Flow_Stop, J4 MultiplexConn, J5 OLED Disp, J6 Press_Sens, J7 MultiplexConn, Q1 Q_NPN_EBC, SW1 SW_DPST, SW2 ~Boot, U1 BLE_FRIEND, U2 PowerButton, U3 LM7805_TO220, U4 HK3FF_RELAY, U5 ADS_1115, U6 Pololu18v17

Commit message: misc
Parts:
- moved G*** 0.51 mm to (76.2, 120.1)
- moved REF** 0.36 mm to (131.1, 119.6)
- moved REF** 0.25 mm to (117.1, 120.7)
Other:
- board text added: "Main Batt"
- board text added: "Main Batt 9-12V when using Greylor PQ-12 gear pump"
- board text removed: "Vbat+"
- board text removed: "Vbat-"
Changed lines of the file:
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@@
   (module MedidoFootprints:BLE_FRIEND (layer F.Cu)
     (at 38.1 60.96 270)
-    (fp_text reference U1 (at 33.02 5.08) (layer F.SilkS)
+    (fp_text reference U1 (at 31.75 12.7) (layer F.SilkS)
       (effects (font (size 1 1) (thickness 0.15)))
     )
@@
   )
   (module MedidoLogo:medidosmall (layer F.Cu)
-    (at 76.2 120.65)
+    (at 76.2 120.142)
     (fp_text reference G*** (at 0 0) (layer F.SilkS) hide
       (effects (font (size 1.524 1.524) (thickness 0.3)))
@@
   )
   (module Symbol:OSHW-Logo2_9.8x8mm_SilkScreen (layer F.Cu)
-    (at 116.84 120.65)
+    (at 117.094 120.65)
     (descr "Open Source Hardware Symbol")
     (tags "Logo Symbol OSHW")
@@
   )
   (module Symbol:KiCad-Logo2_6mm_SilkScreen (layer F.Cu)
-    (at 130.81 119.38)
+    (at 131.064 119.634)
     (descr "KiCad Logo")
     (tags "Logo KiCad")
@@
     (pad 1 np_thru_hole circle (at 0 0) (size 3.2 3.2) (drill 3.2) (layers *.Cu *.Mask))
   )
+  (gr_text "Main Batt 9-12V when using\nGreylor PQ-12 gear pump" (at 100.584 114.046) (layer B.SilkS)
+    (effects (font (size 1.5 1.5) (thickness 0.3)) (justify mirror))
+  )
   (gr_text "Adafruit\nHuzzah\nESP8266\n" (at 93.98 76.2) (layer F.SilkS)
     (effects (font (size 1.016 1.016) (thickness 0.1524)))
@@
     (effects (font (size 1.5 1.5) (thickness 0.3)))
   )
-  (gr_text Vbat- (at 45.72 105.41) (layer F.SilkS)
+  (gr_text "Main Batt" (at 37.084 94.488) (layer F.SilkS)
     (effects (font (size 1.5 1.5) (thickness 0.3)))
   )
-  (gr_text Vbat+ (at 27.94 105.41) (layer F.SilkS)
-    (effects (font (size 1.5 1.5) (thickness 0.3)))
-  )

Commit message: shipped
Parts:
- removed the ? at (180.3, 33.0)
- removed the ? at (25.4, 33.0)
- removed the ? at (25.4, 124.5)
- removed the ? at (180.3, 124.5)
- added ?: MountingHole_3.2mm_M3, MountingHole:MountingHole_3.2mm_M3, F.Cu at (27.9, 35.6)
- added ?: MountingHole_3.2mm_M3, MountingHole:MountingHole_3.2mm_M3, F.Cu at (177.8, 35.6)
- added ?: MountingHole_3.2mm_M3, MountingHole:MountingHole_3.2mm_M3, F.Cu at (177.8, 121.9)
- added ?: MountingHole_3.2mm_M3, MountingHole:MountingHole_3.2mm_M3, F.Cu at (27.9, 121.9)
- moved REF** 1.02 mm to (118.1, 120.7)
- moved G*** 0.57 mm to (76.7, 119.9)
- moved REF** 0.25 mm to (131.3, 119.6)
Routing:
- net Net-(R16-Pad2): vias 1 -> 0
Other:
- board text added: "Run"
- board text added: "Stop boot"
- board text added: "Update"

Commit message: misc
Parts:
- removed ? (x4): MountingHole_3.2mm_M3, MountingHole:MountingHole_3.2mm_M3
- added J8: PwrButton, Connector_PinHeader_2.54mm:PinHeader_1x04_P2.54mm_Vertical, F.Cu at (56.1, 116.3)
- added REF**: MountingHole_3.2mm_M3, MountingHole:MountingHole_3.2mm_M3, F.Cu at (27.9, 35.6)
- added REF**: MountingHole_3.2mm_M3, MountingHole:MountingHole_3.2mm_M3, F.Cu at (177.8, 35.6)
- added REF**: MountingHole_3.2mm_M3, MountingHole:MountingHole_3.2mm_M3, F.Cu at (177.8, 121.9)
- added REF**: MountingHole_3.2mm_M3, MountingHole:MountingHole_3.2mm_M3, F.Cu at (27.9, 121.9)
- moved REF** 3.31 mm to (134.6, 119.9)
- moved REF** 1.30 mm to (119.4, 120.9)
- moved G*** 0.72 mm to (76.2, 119.4)
Routing:
- net Net-(J8-Pad3): track 0.00 -> 38.1 mm, vias 0 -> 1
- net +5V: track 331.9 -> 362.0 mm
- net Net-(J8-Pad4): track 0.00 -> 28.5 mm
- net /OLED_RST: track 129.8 -> 131.5 mm
- net Net-(J7-Pad1): track 35.4 -> 34.8 mm
Other:
- board text added: "Medido Pump UART Rev 3 D. McQueeney 4/2020 FC19"
- board text added: "Power PB"
- board text removed: "Medido Pump UART Rev 2 D. McQueeney 3/2020"

Commit message: misc
Parts:
- removed A1: Adafruit_HUZZAH_ESP8266_breakout, Module:Adafruit_HUZZAH_ESP8266_breakout
- removed the REF** at (134.6, 119.9)
- removed the REF** at (27.9, 35.6)
- removed the REF** at (177.8, 35.6)
- removed the REF** at (177.8, 121.9)
- removed the REF** at (27.9, 121.9)
- removed U4: HK3FF_RELAY, digikey-footprints:Relay_THT_G5LE-14
- removed U5: ADS_1115, MedidoFootprints:ADS_1115
- added ?: MountingHole_3.2mm_M3, MountingHole:MountingHole_3.2mm_M3, F.Cu at (53.3, 55.9)
- added ?: MountingHole_3.2mm_M3, MountingHole:MountingHole_3.2mm_M3, F.Cu at (193.0, 55.9)
- added ?: MountingHole_3.2mm_M3, MountingHole:MountingHole_3.2mm_M3, F.Cu at (193.0, 129.5)
- added ?: MountingHole_3.2mm_M3, MountingHole:MountingHole_3.2mm_M3, F.Cu at (53.3, 129.5)
- added C4: C, Capacitor_THT:C_Disc_D12.0mm_W4.4mm_P7.75mm, F.Cu at (163.8, 99.1)
- added C5: 0.1uF, Capacitor_THT:C_Disc_D12.0mm_W4.4mm_P7.75mm, F.Cu at (113.0, 111.8)
- added D2: 3V Zener, Diode_THT:D_5W_P10.16mm_Horizontal, F.Cu at (156.2, 82.5)
- added Q2: Q_PMOS_GDS, Package_TO_SOT_THT:TO-220-3_Vertical, F.Cu at (88.3, 122.6)
- added R19: 330R, Resistor_THT:R_Axial_DIN0207_L6.3mm_D2.5mm_P10.16mm_Horizontal, F.Cu at (124.5, 113.0)
- added REF**: KiCad-Logo2_5mm_SilkScreen, Symbol:KiCad-Logo2_5mm_SilkScreen, F.Cu at (184.2, 122.6)
- D1: value D -> Power; footprint Diode_THT:D_5W_P10.16mm_Horizontal -> LED_THT:LED_D3.0mm
- Q1: value Q_NPN_EBC -> 2N3904; footprint digikey-footprints:SIP-3_P2.54mm -> Package_TO_SOT_THT:TO-126-3_Vertical
- R11: value 47K -> 100K
- R12: value 4K7 -> 100K
- R13: value 4K7 -> 1K
- R14: value 4K7 -> 33K
- R17: value 3K3 -> 6K8
- SW2: value ~Boot -> On/Off
- U1: value BLE_FRIEND -> Particle_Argon; footprint MedidoFootprints:BLE_FRIEND -> MedidoFootprints:Particle_Argon
- U2: value PowerButton -> HEF4093B; footprint MedidoFootprints:PowerButton -> Package_DIP:DIP-14_W7.62mm
- moved G*** 85.7 mm to (161.9, 121.3)
- moved R14 75.5 mm to (153.7, 118.1), turned to 90 degrees
- moved Q1 75.1 mm to (132.1, 109.2)
- moved R10 71.8 mm to (143.5, 118.1), turned to 90 degrees
- moved D1 66.1 mm to (80.0, 121.3), turned to 0 degrees
- moved R13 64.3 mm to (119.4, 102.9), turned to 270 degrees
- moved R12 62.7 mm to (106.7, 102.9), turned to 270 degrees
- moved C1 61.8 mm to (163.2, 111.8)
- moved J6 61.4 mm to (100.3, 118.1)
- moved R15 61.3 mm to (148.6, 118.1), turned to 90 degrees
- moved U3 56.6 mm to (176.5, 111.8)
- moved J8 55.7 mm to (111.8, 118.1)
- moved C2 54.3 mm to (174.6, 99.7)
- moved U1 52.9 mm to (83.8, 87.6), turned to 90 degrees
- moved REF** 52.6 mm to (172.0, 122.2)
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Connections:
- D1 pad 1: +5V -> GND
- D1 pad 2: GND -> Net-(D1-Pad2)
- J5 pad 3: Net-(A1-Pad16) -> Net-(J5-Pad3)
- J5 pad 4: Net-(A1-Pad15) -> Net-(J5-Pad4)
- J5 pad 5: /OLED_RST -> Net-(J5-Pad5)
- R1 pad 1: Net-(A1-Pad6) -> Net-(R1-Pad1)
- R10 pad 1: +5V -> Net-(R10-Pad1)
- R10 pad 2: Net-(Q1-Pad3) -> GND
- R11 pad 1: /OLED_RST -> Net-(Q2-Pad1)
- R11 pad 2: Net-(Q1-Pad2) -> Net-(J8-Pad3)
- R12 pad 1: +3V3 -> Net-(Q1-Pad3)
- R12 pad 2: Net-(A1-Pad15) -> Net-(C5-Pad1)
- R13 pad 1: +3V3 -> Net-(Q1-Pad2)
- R13 pad 2: Net-(A1-Pad16) -> Net-(R10-Pad1)
- R14 pad 1: Net-(A1-Pad2) -> Net-(R14-Pad1)
- R15 pad 2: Net-(A1-Pad2) -> Net-(R14-Pad1)
- R16 pad 1: Net-(R16-Pad1) -> Net-(C1-Pad1)
- R16 pad 2: Net-(R16-Pad2) -> Net-(D2-Pad1)
- R17 pad 1: Net-(R16-Pad2) -> Net-(D2-Pad1)
- R2 pad 1: Net-(A1-Pad7) -> Net-(R2-Pad1)
- R3 pad 1: Net-(A1-Pad5) -> Net-(R3-Pad1)
- R4 pad 2: Net-(A1-Pad6) -> Net-(R1-Pad1)
- R5 pad 1: Net-(A1-Pad6) -> Net-(R1-Pad1)
- R6 pad 2: Net-(A1-Pad7) -> Net-(R2-Pad1)
- R7 pad 1: Net-(A1-Pad7) -> Net-(R2-Pad1)
- R8 pad 2: Net-(A1-Pad5) -> Net-(R3-Pad1)
- R9 pad 1: Net-(A1-Pad5) -> Net-(R3-Pad1)
- SW1 pad 2: Net-(A1-Pad19) -> +5V
- SW1 pad 3: Net-(SW1-Pad3) -> Net-(SW1-Pad1)
- SW1 pad 4: Net-(A1-Pad20) -> +5V
- SW2 pad 1: +3V3 -> Net-(J8-Pad3)
- SW2 pad 2: Net-(A1-Pad18) -> Net-(J8-Pad4)
- U1 pad 1: Net-(Q1-Pad3) -> Net-(U1-Pad1)
- U1 pad 2: GND -> +3V3
- U1 pad 3: Net-(SW1-Pad1) -> Net-(U1-Pad3)
- U1 pad 4: Net-(SW1-Pad3) -> GND
- U1 pad 5: +5V -> Net-(R14-Pad1)
- U1 pad 6: Net-(U1-Pad6) -> Net-(D2-Pad1)
- U1 pad 7: GND -> Net-(R1-Pad1)
- U1 pad 8: Net-(U1-Pad8) -> Net-(R2-Pad1)
- U2 pad 1: Net-(J4-Pad4) -> GND
- U2 pad 10: Net-(J8-Pad4) -> Net-(Q1-Pad3)
- U2 pad 2: Net-(U2-Pad2) -> GND
- U2 pad 3: GND -> Net-(U2-Pad3)
- U2 pad 4: Net-(A1-Pad18) -> Net-(U2-Pad4)
- U2 pad 5: Net-(U2-Pad5) -> GND
- U2 pad 6: Net-(U2-Pad6) -> GND
- U2 pad 7: Net-(C1-Pad1) -> Net-(U2-Pad7)
- U2 pad 8: Net-(U2-Pad8) -> Net-(J8-Pad3)
- U6 pad 10: Net-(R16-Pad1) -> Net-(C1-Pad1)
- U6 pad 2: Net-(A1-Pad14) -> Net-(U1-Pad25)
- U6 pad 3: Net-(A1-Pad17) -> Net-(U1-Pad24)
- U6 pad 6: Net-(U5-Pad3) -> Net-(U1-Pad10)
- U6 pad 9: Net-(R16-Pad1) -> Net-(C1-Pad1)
Routing:
- net Net-(R14-Pad1): track 0.00 -> 146.1 mm
- net /OLED_RST: track 131.5 -> 0.00 mm, vias 3 -> 0
- net Net-(D2-Pad1): track 0.00 -> 112.4 mm, vias 0 -> 3
- net Net-(J4-Pad4): track 146.1 -> 35.0 mm
- net Net-(R3-Pad1): track 0.00 -> 105.2 mm, vias 0 -> 1
- net Net-(J5-Pad5): track 0.00 -> 98.3 mm, vias 0 -> 4
- net Net-(R1-Pad1): track 0.00 -> 97.3 mm
- net Net-(U1-Pad10): track 0.00 -> 93.0 mm, vias 0 -> 1
- net Net-(A1-Pad16): track 90.8 -> 0.00 mm
- net Net-(C1-Pad1): track 53.7 -> 142.5 mm
- net Net-(J5-Pad3): track 0.00 -> 86.7 mm, vias 0 -> 3
- net Net-(R10-Pad1): track 0.00 -> 78.0 mm, vias 0 -> 4
- net Net-(U1-Pad24): track 0.00 -> 75.0 mm, vias 0 -> 4
- net Net-(U1-Pad25): track 0.00 -> 74.4 mm, vias 0 -> 2
- net Net-(J5-Pad4): track 0.00 -> 74.3 mm
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Other:
- board size 165.1 x 101.6 mm -> 149.9 x 83.8 mm
- board text added: "Int Ext"
- board text added: "Medido Pump Argon Rev 1 D. McQueeney 5/2020"
- board text added: "On/Off"
- board text added: "Press"
- board text removed: "Adafruit Huzzah ESP8266"
- board text removed: "B"
- board text removed: "C"
- board text removed: "E"
- board text removed: "G"
- board text removed: "In"
- board text removed: "K"
- board text removed: "Medido Pump UART Rev 3 D. McQueeney 4/2020 FC19"
- board text removed: "Off"
- board text removed: "Out"
- board text removed: "Press Sens"
- board text removed: "Run"
- board text removed: "Stop boot"
- board text removed: "Update"

Commit message: misc
Parts:
- added JP1: JPF, Jumper:SolderJumper-2_P1.3mm_Open_RoundedPad1.0x1.5mm, F.Cu at (120.7, 66.3)
- added JP2: JPR, Jumper:SolderJumper-2_P1.3mm_Open_RoundedPad1.0x1.5mm, F.Cu at (87.1, 66.3)
- added JP3: JPS, Jumper:SolderJumper-2_P1.3mm_Open_RoundedPad1.0x1.5mm, F.Cu at (153.3, 63.8)
- added R20: 4K7, Resistor_THT:R_Axial_DIN0207_L6.3mm_D2.5mm_P10.16mm_Horizontal, F.Cu at (190.5, 62.2)
- added R21: 4K7, Resistor_THT:R_Axial_DIN0207_L6.3mm_D2.5mm_P10.16mm_Horizontal, F.Cu at (194.3, 62.2)
- moved C3 1.27 mm to (179.1, 67.3)
Connections:
- J8 pad 4: Net-(J8-Pad4) -> Net-(C5-Pad1)
- Q2 pad 2: Net-(J4-Pad4) -> Net-(C1-Pad1)
- Q2 pad 3: Net-(C1-Pad1) -> Net-(J4-Pad4)
- SW2 pad 2: Net-(J8-Pad4) -> Net-(C5-Pad1)
- U2 pad 14: +5V -> Net-(J4-Pad4)
Routing:
- net Net-(C5-Pad1): track 6.88 -> 91.0 mm, vias 0 -> 2
- net Net-(J8-Pad4): track 73.6 -> 0.00 mm, vias 1 -> 0
- net Net-(J4-Pad4): track 35.0 -> 73.0 mm
- net +5V: track 302.5 -> 265.7 mm, vias 2 -> 0
- net Net-(J5-Pad4): track 74.3 -> 96.9 mm
- net Net-(J5-Pad3): track 86.7 -> 106.6 mm
- net +3V3: track 143.6 -> 159.7 mm
- net Net-(J3-Pad1): track 16.8 -> 26.4 mm
- net Net-(JP1-Pad2): track 97.3 -> 103.1 mm
- net Net-(JP2-Pad2): track 52.7 -> 58.3 mm
- net Net-(JP3-Pad2): track 105.2 -> 110.7 mm
- net Net-(J2-Pad1): track 15.5 -> 18.7 mm
- net Net-(J1-Pad1): track 15.5 -> 18.6 mm
- net Net-(Q1-Pad2): track 16.6 -> 17.9 mm
- net Net-(C1-Pad1): track 142.5 -> 143.5 mm
Other:
- board text added: "Medido Pump Argon Rev 2 D. McQueeney 6/2020"
- board text removed: "Medido Pump Argon Rev 1 D. McQueeney 5/2020"

Commit message: misc
Parts:
- added C6: 0.1 uF, Capacitor_THT:C_Disc_D12.0mm_W4.4mm_P7.75mm, F.Cu at (107.8, 57.1)
- added C7: 0.1 uF, Capacitor_THT:C_Disc_D12.0mm_W4.4mm_P7.75mm, F.Cu at (82.5, 57.1)
- added C8: 0.1 uF, Capacitor_THT:C_Disc_D12.0mm_W4.4mm_P7.75mm, F.Cu at (141.0, 57.1)
- added J9: Aux I/O, Connector_PinHeader_2.54mm:PinHeader_1x08_P2.54mm_Vertical, F.Cu at (53.3, 102.9)
- added R22: 100K, Resistor_THT:R_Axial_DIN0207_L6.3mm_D2.5mm_P10.16mm_Horizontal, F.Cu at (125.1, 57.1)
- added R23: 100K, Resistor_THT:R_Axial_DIN0207_L6.3mm_D2.5mm_P10.16mm_Horizontal, F.Cu at (90.2, 57.1)
- added R24: 100K, Resistor_THT:R_Axial_DIN0207_L6.3mm_D2.5mm_P10.16mm_Horizontal, F.Cu at (156.8, 57.1)
- added R25: 10K, Resistor_THT:R_Axial_DIN0207_L6.3mm_D2.5mm_P10.16mm_Horizontal, F.Cu at (74.3, 116.2)
Connections:
- U1 pad 11: Net-(U1-Pad11) -> SCK
- U1 pad 12: Net-(U1-Pad12) -> MOSI
- U1 pad 13: Net-(U1-Pad13) -> MISO
- U1 pad 19: Net-(U1-Pad19) -> D2
- U1 pad 20: Net-(U1-Pad20) -> D3
- U1 pad 21: Net-(U1-Pad21) -> D4
- U1 pad 7: Net-(JP1-Pad2) -> Net-(C6-Pad1)
- U1 pad 8: Net-(JP2-Pad2) -> Net-(C7-Pad1)
- U1 pad 9: Net-(JP3-Pad2) -> Net-(C8-Pad1)
Routing:
- net Net-(C8-Pad1): track 0.00 -> 102.6 mm, vias 0 -> 2
- net Net-(C6-Pad1): track 0.00 -> 99.1 mm, vias 0 -> 3
- net Net-(JP3-Pad2): track 110.7 -> 28.6 mm
- net D4: track 0.00 -> 75.7 mm, vias 0 -> 3
- net Net-(JP1-Pad2): track 103.1 -> 31.1 mm, vias 0 -> 1
- net Net-(C7-Pad1): track 0.00 -> 70.6 mm, vias 0 -> 5
- net D2: track 0.00 -> 65.9 mm, vias 0 -> 3
- net MOSI: track 0.00 -> 63.2 mm, vias 0 -> 3
- net D3: track 0.00 -> 60.8 mm, vias 0 -> 6
- net MISO: track 0.00 -> 56.1 mm, vias 0 -> 4
- net SCK: track 0.00 -> 50.3 mm, vias 0 -> 1
- net +3V3: track 159.7 -> 204.6 mm
- net Net-(JP2-Pad2): track 58.3 -> 28.3 mm
- net Net-(J4-Pad4): track 73.0 -> 94.4 mm, vias 0 -> 1
- net Net-(Q2-Pad1): track 39.1 -> 54.2 mm
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Other:
- board text added: "Medido Pump Argon Rev 3 D. McQueeney 2/2021"
- board text removed: "Medido Pump Argon Rev 2 D. McQueeney 6/2020"
