File: MedidoPump.sch (KiCad schematic (older format))
At the start: 39 parts, among them J1 Flow_Fwd, J2 Flow_Rev, J3 Flow_Stop, J4 MultiplexConn, J5 OLED Disp, J6 Press_Sens, J7 MultiplexConn, Q1 Q_NPN_EBC, SW1 SW_DPST, SW2 ~Boot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

Commit message: shipped
Other:
- note added: "Note: For BioTech sensors (open collector), replace R1,R2,R3 with \nwires and set R4,R6,R8 to 2K2. For Digitech's sensors (active output), omit R4,R6,R8\n"
- moved on the sheet: R18, U6
Changed lines of the file:
@@
 Sheet 1 1
 Title "Medido Pump"
-Date ""
+Date "2020-03-20"
 Rev "2.0"
-Comp ""
+Comp "DFM"
 Comment1 ""
 Comment2 ""
@@
 	5150 2100 5150 700
 Wire Wire Line
-	5150 700  6550 700
-Wire Wire Line
-	6550 700  6550 1600
+	5150 700  6500 700
+Wire Wire Line
+	6500 700  6500 1600
 Wire Wire Line
 	4250 1600 5050 1600
@@
 L medido:Pololu18v17 U6
 U 1 1 5E759E1D
-P 7350 1850
-F 0 "U6" V 6735 1850 50  0000 C CNN
-F 1 "Pololu18v17" V 6826 1850 50  0000 C CNN
-F 2 "MedidoFootprints:Pololu18V17" H 7250 1750 50  0001 C CNN
-F 3 "" H 7250 1750 50  0001 C CNN
-	1    7350 1850
+P 7300 1850
+F 0 "U6" V 6685 1850 50  0000 C CNN
+F 1 "Pololu18v17" V 6776 1850 50  0000 C CNN
+F 2 "MedidoFootprints:Pololu18V17" H 7200 1750 50  0001 C CNN
+F 3 "" H 7200 1750 50  0001 C CNN
+	1    7300 1850
 	0    1    1    0
 $EndComp
@@
 	5500 3200 5500 3850
 Wire Wire Line
-	6550 1600 6800 1600
-Wire Wire Line
-	6450 1700 6800 1700
-Wire Wire Line
-	6300 3200 8100 3200
-Wire Wire Line
-	8100 3200 8100 2200
-Wire Wire Line
-	8100 2200 7900 2200
+	6500 1600 6750 1600
+Wire Wire Line
+	6300 3200 8050 3200
+Wire Wire Line
+	8050 3200 8050 2200
+Wire Wire Line
+	8050 2200 7850 2200
 Connection ~ 6300 3200
 Wire Wire Line
-	7900 2100 8100 2100
-Wire Wire Line
-	8100 2100 8100 2200
-Connection ~ 8100 2200
+	7850 2100 8050 2100
+Wire Wire Line
+	8050 2100 8050 2200
+Connection ~ 8050 2200
 $Comp
 L power:GND #PWR043
 U 1 1 5E77CAFD
-P 7200 2500
-F 0 "#PWR043" H 7200 2250 50  0001 C CNN
-F 1 "GND" H 7205 2327 50  0000 C CNN
-F 2 "" H 7200 2500 50  0001 C CNN
-F 3 "" H 7200 2500 50  0001 C CNN
-	1    7200 2500
+P 7150 2500
+F 0 "#PWR043" H 7150 2250 50  0001 C CNN
+F 1 "GND" H 7155 2327 50  0000 C CNN
+F 2 "" H 7150 2500 50  0001 C CNN
+F 3 "" H 7150 2500 50  0001 C CNN
+	1    7150 2500
 	1    0    0    -1
 $EndComp
@@
 L power:GND #PWR044
 U 1 1 5E77CB8E
-P 7350 2500
-F 0 "#PWR044" H 7350 2250 50  0001 C CNN
-F 1 "GND" H 7355 2327 50  0000 C CNN
-F 2 "" H 7350 2500 50  0001 C CNN
-F 3 "" H 7350 2500 50  0001 C CNN
-	1    7350 2500
+P 7300 2500
+F 0 "#PWR044" H 7300 2250 50  0001 C CNN
+F 1 "GND" H 7305 2327 50  0000 C CNN
+F 2 "" H 7300 2500 50  0001 C CNN
+F 3 "" H 7300 2500 50  0001 C CNN
+	1    7300 2500
 	1    0    0    -1
 $EndComp
@@
 L power:GND #PWR045
 U 1 1 5E77CC1F
-P 7500 2500
-F 0 "#PWR045" H 7500 2250 50  0001 C CNN
-F 1 "GND" H 7505 2327 50  0000 C CNN
-F 2 "" H 7500 2500 50  0001 C CNN
-F 3 "" H 7500 2500 50  0001 C CNN
-	1    7500 2500
+P 7450 2500
+F 0 "#PWR045" H 7450 2250 50  0001 C CNN
+F 1 "GND" H 7455 2327 50  0000 C CNN
+F 2 "" H 7450 2500 50  0001 C CNN
+F 3 "" H 7450 2500 50  0001 C CNN
+	1    7450 2500
 	1    0    0    -1
 $EndComp
@@
 Wire Wire Line
 	6300 1700 6300 2000
-Wire Wire Line
-	6300 2000 6800 2000
-NoConn ~ 6800 1800
-NoConn ~ 6800 1900
-NoConn ~ 6800 2100
-NoConn ~ 6800 2200
-Wire Wire Line
-	7900 1800 8050 1800
-Wire Wire Line
-	7900 1700 8050 1700
-Wire Wire Line
-	8050 1700 8050 1800
-Wire Wire Line
-	7900 2000 8050 2000
-Wire Wire Line
-	7900 1900 8050 1900
-Wire Wire Line
-	8050 1900 8050 2000
+NoConn ~ 6750 1800
+NoConn ~ 6750 1900
+NoConn ~ 6750 2100
+NoConn ~ 6750 2200
+Wire Wire Line
+	7850 1800 8000 1800
+Wire Wire Line
+	7850 1700 8000 1700
+Wire Wire Line
+	8000 1700 8000 1800
+Wire Wire Line
+	7850 2000 8000 2000
+Wire Wire Line
+	7850 1900 8000 1900
+Wire Wire Line
+	8000 1900 8000 2000
 Text Notes 9150 1700 0    50   ~ 0
 Mot B
@@
 L Device:R_Small_US R18
 U 1 1 5E7AD3CB
-P 8000 1500
-F 0 "R18" V 7795 1500 50  0000 C CNN
-F 1 "Curr Lim" V 7886 1500 50  0000 C CNN
-F 2 "Resistor_THT:R_Axial_DIN0207_L6.3mm_D2.5mm_P10.16mm_Horizontal" H 8000 1500 50  0001 C CNN
-F 3 "" H 8000 1500 50  0001 C CNN
-	1    8000 1500
+P 7950 1500
+F 0 "R18" V 7745 1500 50  0000 C CNN
+F 1 "Curr Lim" V 7836 1500 50  0000 C CNN
+F 2 "Resistor_THT:R_Axial_DIN0207_L6.3mm_D2.5mm_P10.16mm_Horizontal" H 7950 1500 50  0001 C CNN
+F 3 "" H 7950 1500 50  0001 C CNN
+	1    7950 1500
 	0    1    1    0
 $EndComp
 Wire Wire Line
-	7900 1600 8250 1600
-Wire Wire Line
-	8250 1600 8250 1500
-Wire Wire Line
-	8250 1500 8100 1500
+	7850 1600 8200 1600
+Wire Wire Line
+	8200 1600 8200 1500
+Wire Wire Line
+	8200 1500 8050 1500
 NoConn ~ 5300 3750
 Wire Wire Line
-	8500 1800 8050 1800
-Connection ~ 8050 1800
-Wire Wire Line
-	8500 1900 8050 1900
-Connection ~ 8050 1900
+	8500 1800 8000 1800
+Connection ~ 8000 1800
+Wire Wire Line
+	8500 1900 8000 1900
+Connection ~ 8000 1900
 Wire Wire Line
 	1900 3700 1900 3800
@@
 	9100 2350 9100 2050
 Connection ~ 8800 2350
+Text Notes 2450 7450 0    50   ~ 0
+Note: For BioTech sensors (open collector), replace R1,R2,R3 with \nwires and set R4,R6,R8 to 2K2. For Digitech's sensors (active output), omit R4,R6,R8\n
+Wire Wire Line
+	6300 2000 6750 2000
+Wire Wire Line
+	6450 1700 6750 1700
 $EndSCHEMATC

Commit message: misc
Parts:
- removed U2: PowerButton, MedidoFootprints:PowerButton, symbol MedidoPump-rescue:PowerButton-medido
- added J8: PwrButton, Connector_PinHeader_2.54mm:PinHeader_1x04_P2.54mm_Vertical, symbol Connector:Conn_01x04_Male
- added U2: PowerButton, MedidoFootprints:PowerButton, symbol medido:PowerButton
Connections:
- wire segments 158 -> 169
Other:
- note added: "+5"
- note added: "Note: R18 opt curr lim resistor to be monuted \non 18v17 or via addl pins and mounted on board."
- note added: "S1"
- note added: "S3"
Changed lines of the file:
@@
 Title "Medido Pump"
 Date "2020-03-20"
-Rev "2.0"
+Rev "3.0"
 Comp "DFM"
 Comment1 ""
@@
 Wire Wire Line
 	4450 1800 4450 5200
-Text Notes 6500 5700 0    50   ~ 0
+Text Notes 6750 5950 0    50   ~ 0
 Blk
-Text Notes 6500 5800 0    50   ~ 0
+Text Notes 6750 6050 0    50   ~ 0
 Red
-Text Notes 6500 5900 0    50   ~ 0
+Text Notes 6750 6150 0    50   ~ 0
 Wht
 Wire Wire Line
@@
 F 3 "" H 3450 1000 50  0001 C CNN
 	1    3450 1000
-	1    0    0    -1
-$EndComp
-$Comp
-L MedidoPump-rescue:PowerButton-medido U2
-U 1 1 5E6F1000
-P 2600 3850
-F 0 "U2" H 2550 3450 50  0000 L CNN
-F 1 "PowerButton" H 2400 3350 50  0000 L CNN
-F 2 "MedidoFootprints:PowerButton" H 2350 3750 50  0001 C CNN
-F 3 "" H 2350 3750 50  0001 C CNN
-	1    2600 3850
 	1    0    0    -1
 $EndComp
@@
 Wire Wire Line
 	6450 1700 6750 1700
+$Comp
+L Connector:Conn_01x04_Male J8
+U 1 1 5E8A686A
+P 5150 5800
+F 0 "J8" H 5250 6000 50  0000 R CNN
+F 1 "PwrButton" H 5400 6100 50  0000 R CNN
+F 2 "Connector_PinHeader_2.54mm:PinHeader_1x04_P2.54mm_Vertical" H 5150 5800 50  0001 C CNN
+F 3 "~" H 5150 5800 50  0001 C CNN
+	1    5150 5800
+	-1   0    0    1
+$EndComp
+Text Notes 5250 5950 0    50   ~ 0
+Gnd
+Text Notes 5250 5850 0    50   ~ 0
++5
+Text Notes 5250 5750 0    50   ~ 0
+S1
+Text Notes 5250 5650 0    50   ~ 0
+S3
+Wire Wire Line
+	4950 5900 4700 5900
+Wire Wire Line
+	4700 5900 4700 5950
+$Comp
+L power:GND #PWR047
+U 1 1 5E8C844A
+P 4700 5950
+F 0 "#PWR047" H 4700 5700 50  0001 C CNN
+F 1 "GND" H 4705 5777 50  0000 C CNN
+F 2 "" H 4700 5950 50  0001 C CNN
+F 3 "" H 4700 5950 50  0001 C CNN
+	1    4700 5950
+	1    0    0    -1
+$EndComp
+Wire Wire Line
+	4950 5800 4500 5800
+Wire Wire Line
+	4500 5800 4500 5700
+$Comp
+L power:+5V #PWR046
+U 1 1 5E8CF33F
+P 4500 5700
+F 0 "#PWR046" H 4500 5550 50  0001 C CNN
+F 1 "+5V" H 4515 5873 50  0000 C CNN
+F 2 "" H 4500 5700 50  0001 C CNN
+F 3 "" H 4500 5700 50  0001 C CNN
+	1    4500 5700
+	1    0    0    -1
+$EndComp
+$Comp
+L medido:PowerButton U2
+U 1 1 5E8E42C3
+P 2600 3850
+F 0 "U2" H 2600 4265 50  0000 C CNN
+F 1 "PowerButton" H 2600 4174 50  0000 C CNN
+F 2 "MedidoFootprints:PowerButton" H 2350 3750 50  0001 C CNN
+F 3 "" H 2350 3750 50  0001 C CNN
+	1    2600 3850
+	1    0    0    -1
+$EndComp
+Wire Wire Line
+	2700 4300 2700 5300
+Wire Wire Line
+	2700 5300 4950 5300
+Wire Wire Line
+	4950 5300 4950 5600
+Wire Wire Line
+	2600 4300 2600 5350
+Wire Wire Line
+	2600 5350 4900 5350
+Wire Wire Line
+	4900 5350 4900 5700
+Wire Wire Line
+	4900 5700 4950 5700
+Text Notes 7750 2650 0    50   ~ 0
+Note: R18 opt curr lim resistor to be monuted \non 18v17 or via addl pins and mounted on board.
 $EndSCHEMATC

Commit message: misc
Parts:
- removed A1: Adafruit_HUZZAH_ESP8266_breakout, Module:Adafruit_HUZZAH_ESP8266_breakout, symbol MCU_Module:Adafruit_HUZZAH_ESP8266_breakout
- removed D1: D, Diode_THT:D_5W_P10.16mm_Horizontal, symbol Device:D
- removed U1: BLE_FRIEND, MedidoFootprints:BLE_FRIEND, symbol medido:BLE_FRIEND
- removed U2: PowerButton, MedidoFootprints:PowerButton, symbol medido:PowerButton
- removed U4: HK3FF_RELAY, digikey-footprints:Relay_THT_G5LE-14, symbol MedidoPump-rescue:HK3FF_RELAY-medido
- removed U5: ADS_1115, MedidoFootprints:ADS_1115, symbol medido:ADS_1115
- added C4: C, Capacitor_THT:C_Disc_D12.0mm_W4.4mm_P7.75mm, symbol Device:C
- added C5: 0.1uF, Capacitor_THT:C_Disc_D12.0mm_W4.4mm_P7.75mm, symbol Device:C
- added D1: Power, LED_THT:LED_D3.0mm, symbol Device:LED_Small
- added D2: 3V Zener, Diode_THT:D_5W_P10.16mm_Horizontal, symbol Device:D_Zener
- added Q2: Q_PMOS_GDS, Package_TO_SOT_THT:TO-220-3_Vertical, symbol Device:Q_PMOS_GDS
- added R19: 330R, Resistor_THT:R_Axial_DIN0207_L6.3mm_D2.5mm_P10.16mm_Horizontal, symbol Device:R_Small_US
- added U1: Particle_Argon, MedidoFootprints:Particle_Argon, symbol medido:Particle_Argon
- added U2: HEF4093B, Package_DIP:DIP-14_W7.62mm, symbol 4xxx:HEF4093B
- Q1: value Q_NPN_EBC -> 2N3904; footprint digikey-footprints:SIP-3_P2.54mm -> Package_TO_SOT_THT:TO-126-3_Vertical
- R11: value 47K -> 100K
- R12: value 4K7 -> 100K
- R13: value 4K7 -> 1K
- R14: value 4K7 -> 33K
- R17: value 3K3 -> 6K8
- SW2: value ~Boot -> On/Off
Connections:
- net +3V3: now also U1.2 (3V3); no longer R12.1, R13.1, SW2.1
- net +5V: now also SW1.2, SW1.4, C4.1, R19.2, U2.14 (VCC); no longer R10.1
- net GND: now also R10.2, C4.2, C5.2, D1.1 (K), D2.2 (A), U1.4 (Gnd), U2.1, U2.2, U2.5, U2.6
- net at U6.2 (Dir): now also U1.25 (D8)
- net at J5.4 (Pin_4): now also U1.17 (SDA); no longer R12.2
- net at J5.3 (Pin_3): now also U1.18 (SCL); no longer R13.2
- net at U6.3 (PWM): now also U1.24 (D7)
- net at SW2.2: now also J8.4 (Pin_4)
- net at R14.1, R15.2: now also U1.5 (A0)
- net at R3.1, R8.2, R9.1: now also U1.9 (A4)
- net at R1.1, R4.2, R5.1: now also U1.7 (A2)
- net at R2.1, R6.2, R7.1: now also U1.8 (A3)
- net at Q1.3 (C): now also R12.1, U2.10, U2.12, U2.13; no longer R10.2
- net at SW1.1: now also SW1.3, U1.26 (VBUS)
- net at C1.1, U3.1 (VI): now also R16.1, U6.10 (Vin), U6.9 (Vin), Q2.3 (S)
- net at R11.2: now also J8.3 (Pin_3), SW2.1, U2.8, U2.9; no longer Q1.2 (B)
- net at R16.2, R17.1: now also D2.1 (K), U1.6 (A1)
- net at U6.6 (CS): now also U1.10 (A5)
- net at J4.4 (P4), J4.5 (P5), J4.6 (P6): now also Q2.2 (D)
- net OLED_RST: no longer names the net of J5.5 (Pin_5)
- net OLED_RST: now also U1.23 (D6); no longer R11.1
- new net: R10.1, R13.2, U1.22 (D5)
- new net: Q2.1 (G), R11.1, U2.11
- new net: C5.1, R12.2
- new net: Q1.2 (B), R13.1
- new net: D1.2 (A), R19.1
- no-connect marks 16 -> 17
Other:
- moved on the sheet: J8

Commit message: misc
Parts:
- added JP1: JPF, Jumper:SolderJumper-2_P1.3mm_Open_RoundedPad1.0x1.5mm, symbol Jumper:SolderJumper_2_Open
- added JP2: JPR, Jumper:SolderJumper-2_P1.3mm_Open_RoundedPad1.0x1.5mm, symbol Jumper:SolderJumper_2_Open
- added JP3: JPS, Jumper:SolderJumper-2_P1.3mm_Open_RoundedPad1.0x1.5mm, symbol Jumper:SolderJumper_2_Open
- added R20, R21: 4K7, Resistor_THT:R_Axial_DIN0207_L6.3mm_D2.5mm_P10.16mm_Horizontal, symbol Device:R_Small_US
Connections:
- net +3V3: now also R20.1, R21.1
- net +5V: no longer U2.14 (VCC)
- net at C1.1, R16.1, U3.1 (VI)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: now also Q2.2 (D); no longer Q2.3 (S)
- net at J1.1 (Pin_1), R1.2: now also JP1.1 (A)
- net at J2.1 (Pin_1), R2.2: now also JP2.1 (A)
- net at J3.1 (Pin_1), R3.2: now also JP3.1 (A)
- net at R1.1, R4.2, R5.1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: now also JP1.2 (B)
- net at R2.1, R6.2, R7.1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: now also JP2.2 (B)
- net at R3.1, R8.2, R9.1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: now also JP3.2 (B)
- net at J5.3 (Pin_3), U1.18 (SCL): now also R20.2
- net at J5.4 (Pin_4), U1.17 (SDA): now also R21.2
- net at J4.4 (P4), J4.5 (P5), J4.6 (P6): now also Q2.3 (S), U2.14 (VCC); no longer Q2.2 (D)
- net at J8.4 (Pin_4), SW2.2: now also C5.1, R12.2
Other:
- note added: "I2C Pullups"
- moved on the sheet: C5
Changed lines of the file:
@@
 Title "Medido Pump / Particle Argon"
 Date "2020-03-20"
-Rev "1.0"
+Rev "2.0"
 Comp "DFM"
 Comment1 ""
@@
 	4200 1950 4950 1950
 Wire Wire Line
-	6050 2650 6050 4800
+	6050 2650 6050 4000
 Wire Wire Line
 	6050 4800 6250 4800
@@
 	6050 2550 6200 2550
 Wire Wire Line
-	6200 2550 6200 4600
+	6200 2550 6200 4050
 Wire Wire Line
 	6200 4600 5850 4600
@@
 Wire Wire Line
 	6300 3100 5950 3100
-Wire Wire Line
-	5950 3100 5950 4700
 Wire Wire Line
 	5950 4700 6250 4700
@@
 L Device:C C5
 U 1 1 5ED5F57F
-P 1600 1650
-F 0 "C5" H 1715 1696 50  0000 L CNN
-F 1 "0.1uF" H 1715 1605 50  0000 L CNN
-F 2 "Capacitor_THT:C_Disc_D12.0mm_W4.4mm_P7.75mm" H 1638 1500 50  0001 C CNN
-F 3 "~" H 1600 1650 50  0001 C CNN
-	1    1600 1650
+P 1600 1700
+F 0 "C5" H 1715 1746 50  0000 L CNN
+F 1 "0.1uF" H 1715 1655 50  0000 L CNN
+F 2 "Capacitor_THT:C_Disc_D12.0mm_W4.4mm_P7.75mm" H 1638 1550 50  0001 C CNN
+F 3 "~" H 1600 1700 50  0001 C CNN
+	1    1600 1700
 	1    0    0    -1
 $EndComp
@@
 Wire Wire Line
 	2550 850  2550 1250
-Wire Wire Line
-	1600 1550 1300 1550
 $Comp
 L Switch:SW_Push SW2
@@
 	1    0    0    -1
 $EndComp
-Wire Wire Line
-	1600 1800 1600 1950
 $Comp
 L Device:R_Small_US R13
@@
 Connection ~ 2550 1250
 Wire Wire Line
-	3250 950  3350 950
-Wire Wire Line
 	6600 800  6600 1000
 Wire Wire Line
@@
 	1    0    0    -1
 $EndComp
-$Comp
-L power:+5V #PWR024
-U 1 1 5EE3F7B0
-P 2500 2150
-F 0 "#PWR024" H 2500 2000 50  0001 C CNN
-F 1 "+5V" H 2515 2323 50  0000 C CNN
-F 2 "" H 2500 2150 50  0001 C CNN
-F 3 "" H 2500 2150 50  0001 C CNN
-	1    2500 2150
-	1    0    0    -1
-$EndComp
 Wire Wire Line
 	2600 3950 2600 4350
@@
 Wire Wire Line
 	1300 2050 1300 1550
-Connection ~ 1300 1550
 Wire Wire Line
 	1300 1550 1250 1550
-Wire Wire Line
-	3350 950  3350 3450
 Connection ~ 3350 3800
 Wire Wire Line
@@
 Wire Wire Line
 	2450 1750 3150 1750
-Wire Wire Line
-	2850 950  2850 3800
 Wire Wire Line
 	2850 3800 1490 3800
@@
 Wire Wire Line
 	4700 3200 6300 3200
-Connection ~ 3350 3450
 Wire Wire Line
 	3350 3450 3350 3800
@@
 Wire Wire Line
 	4850 3800 4850 3900
+$Comp
+L Device:R_Small_US R20
+U 1 1 5EEF73E9
+P 5450 3800
+F 0 "R20" H 5518 3846 50  0000 L CNN
+F 1 "4K7" H 5518 3755 50  0000 L CNN
+F 2 "Resistor_THT:R_Axial_DIN0207_L6.3mm_D2.5mm_P10.16mm_Horizontal" H 5450 3800 50  0001 C CNN
+F 3 "~" H 5450 3800 50  0001 C CNN
+	1    5450 3800
+	1    0    0    -1
+$EndComp
+$Comp
+L Device:R_Small_US R21
+U 1 1 5EEF74AA
+P 5700 3800
+F 0 "R21" H 5768 3846 50  0000 L CNN
+F 1 "4K7" H 5768 3755 50  0000 L CNN
+F 2 "Resistor_THT:R_Axial_DIN0207_L6.3mm_D2.5mm_P10.16mm_Horizontal" H 5700 3800 50  0001 C CNN
+F 3 "~" H 5700 3800 50  0001 C CNN
+	1    5700 3800
+	1    0    0    -1
+$EndComp
+$Comp
+L power:+3V3 #PWR0101
+U 1 1 5EEF7739
+P 5450 3700
+F 0 "#PWR0101" H 5450 3550 50  0001 C CNN
+F 1 "+3V3" H 5465 3873 50  0000 C CNN
+F 2 "" H 5450 3700 50  0001 C CNN
+F 3 "" H 5450 3700 50  0001 C CNN
+	1    5450 3700
+	1    0    0    -1
+$EndComp
+Wire Wire Line
+	5450 3700 5700 3700
+Connection ~ 5450 3700
+Wire Wire Line
+	5700 3900 5700 4000
+Wire Wire Line
+	5700 4000 6050 4000
+Connection ~ 6050 4000
+Wire Wire Line
+	6050 4000 6050 4800
+Wire Wire Line
+	5450 3900 5450 4050
+Wire Wire Line
+	5950 3100 5950 4700
+Wire Wire Line
+	5450 4050 6200 4050
+Connection ~ 6200 4050
+Wire Wire Line
+	6200 4050 6200 4600
+Text Notes 5400 4200 0    50   ~ 0
+I2C Pullups
+Wire Wire Line
+	1600 1550 1600 1500
+Wire Wire Line
+	1600 1850 1600 1950
+Wire Wire Line
+	1300 1550 1600 1550
+Connection ~ 1300 1550
+Connection ~ 1600 1550
+Wire Wire Line
+	2500 2150 2850 2150
+Wire Wire Line
+	2850 2150 2850 3800
+Wire Wire Line
+	2850 950  2850 1600
+Wire Wire Line
+	2850 1600 3350 1600
+Wire Wire Line
+	3350 1600 3350 3450
+Connection ~ 3350 3450
+Wire Wire Line
+	3250 950  3250 2150
+Wire Wire Line
+	3250 2150 2850 2150
+Connection ~ 2850 2150
+$Comp
+L Jumper:SolderJumper_2_Open JP1
+U 1 1 5ED659D2
+P 1700 5400
+F 0 "JP1" V 1654 5468 50  0000 L CNN
+F 1 "JPF" V 1745 5468 50  0000 L CNN
+F 2 "Jumper:SolderJumper-2_P1.3mm_Open_RoundedPad1.0x1.5mm" H 1700 5400 50  0001 C CNN
+F 3 "~" H 1700 5400 50  0001 C CNN
+	1    1700 5400
+	0    1    1    0
+$EndComp
+Wire Wire Line
+	1700 5200 1700 5250
+Connection ~ 1700 5200
+Wire Wire Line
+	1700 5550 1900 5550
+Wire Wire Line
+	1900 5550 1900 5200
+Connection ~ 1900 5200
+$Comp
+L Jumper:SolderJumper_2_Open JP2
+U 1 1 5ED7A057
+P 1700 6300
+F 0 "JP2" V 1654 6368 50  0000 L CNN
+F 1 "JPR" V 1745 6368 50  0000 L CNN
+F 2 "Jumper:SolderJumper-2_P1.3mm_Open_RoundedPad1.0x1.5mm" H 1700 6300 50  0001 C CNN
+F 3 "~" H 1700 6300 50  0001 C CNN
+	1    1700 6300
+	0    1    1    0
+$EndComp
+$Comp
+L Jumper:SolderJumper_2_Open JP3
+U 1 1 5ED7A250
+P 1700 7350
+F 0 "JP3" V 1654 7418 50  0000 L CNN
+F 1 "JPS" V 1745 7418 50  0000 L CNN
+F 2 "Jumper:SolderJumper-2_P1.3mm_Open_RoundedPad1.0x1.5mm" H 1700 7350 50  0001 C CNN
+F 3 "~" H 1700 7350 50  0001 C CNN
+	1    1700 7350
+	0    1    1    0
+$EndComp
+Wire Wire Line
+	1700 6150 1700 6100
+Connection ~ 1700 6100
+Wire Wire Line
+	1700 6450 1900 6450
+Wire Wire Line
+	1900 6450 1900 6100
+Connection ~ 1900 6100
+Wire Wire Line
+	1700 7200 1700 7150
+Connection ~ 1700 7150
+Wire Wire Line
+	1700 7500 1900 7500
+Wire Wire Line
+	1900 7500 1900 7150
+Connection ~ 1900 7150
 $EndSCHEMATC
