File: NewMC/NewMC/NewMC.kicad_pcb (KiCad board)
At the start: 2 copper layers, 22.2 x 34.9 mm, 3 parts, among them U1 Pololu18v17, U2 IFX9201SGAUMA1

Commit message: misc
Parts:
- added C3: CP1, Capacitor_THT:CP_Radial_D6.3mm_P2.50mm, F.Cu at (81.9, 94.0)
- added D1: D_Zener 3.3V, Diode_THT:D_DO-41_SOD81_P2.54mm_Vertical_KathodeUp, F.Cu at (76.2, 95.2)
- added R1: 1K, Resistor_THT:R_Axial_DIN0207_L6.3mm_D2.5mm_P2.54mm_Vertical, F.Cu at (74.3, 78.1)
- added U3: L4931 3.3V Reg, Package_TO_SOT_THT:TO-92_Inline, F.Cu at (87.6, 80.6)
Routing:
- net Net-(C3-Pad1): track 0.00 -> 40.2 mm, vias 0 -> 1
- net Net-(C1-Pad1): track 50.3 -> 61.1 mm
Other:
- board text added: "IFX9201 R2 02/2021 McQ"
- board text removed: "IFX9201 Test 07/2020 McQ"

Commit message: misc
Other:
- net class Default removed
